File: 2.设计资料/2.硬件电路/第一章放大电路/第一章放大电路.sch (KiCad schematic (older format))
At the start: 110 parts, among them J1 VIN_15V, J10 Vout4-, J11 Vout4+, J12 Vout5, J13 Vin_sin7, J14 Vin_sin6, J15 Vin_sin8, J16 Vout7, J17 Vout6, J18 Vout8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

Commit message: PCB 布局完成
Parts:
- D1: value D_Small -> 1N4148
Other:
- moved on the sheet: C11, C13, C4, C9, J3, J5, Q2, R3, R4, R7, R8
